File: Hardware/PCB/Leveller.kicad_pcb (KiCad board)
At the start: 2 copper layers, 20 x 27.8 mm, 32 parts, among them J12 Conn_01x06_Socket, J7 Conn_01x05_Pin, U1 TL074, U2 TL074

Commit message: Version 1.0 of hardware ordered
Parts:
- removed J12: Conn_01x06_Socket, Connector_PinSocket_2.54mm:PinSocket_1x06_P2.54mm_Vertical
- removed J7: Conn_01x05_Pin, Connector_PinSocket_2.54mm:PinSocket_1x05_P2.54mm_Vertical
- added C4: 10uF, Capacitor_SMD:CP_Elec_4x5.4, F.Cu at (63.0, 44.2)
- added C6: 10uF, Capacitor_SMD:CP_Elec_4x5.4, F.Cu at (63.0, 51.1)
- added D1: 1N5819, Diode_SMD:D_SOD-123, F.Cu at (57.0, 55.8)
- added D4: 1N5819, Diode_SMD:D_SOD-123, F.Cu at (66.8, 52.0)
- added FB1: FerriteBead, Resistor_SMD:R_0603_1608Metric, F.Cu at (57.8, 58.1)
- added FB2: FerriteBead, Resistor_SMD:R_0603_1608Metric, F.Cu at (66.0, 55.3)
- added J13: Audio to Daisy, connect to J13, Connector_PinHeader_2.54mm:PinHeader_1x03_P2.54mm_Vertical, F.Cu at (52.5, 79.4)
- added J14: Audio from Daisy, connect to J10, Connector_PinHeader_2.54mm:PinHeader_1x03_P2.54mm_Vertical, F.Cu at (67.5, 79.4)
- added J17: Audio output, connect to J16, Connector_PinHeader_2.54mm:PinHeader_1x03_P2.54mm_Vertical, F.Cu at (51.8, 42.1)
- added J18: Audio input, connect to J15, Connector_PinHeader_2.54mm:PinHeader_1x03_P2.54mm_Vertical, F.Cu at (68.2, 42.1)
- added J6: Eurorack_Power, Connector_PinHeader_2.54mm:PinHeader_2x05_P2.54mm_Vertical, B.Cu at (55.4, 52.7)
- moved C2 14.0 mm to (64.8, 77.1), turned to 90 degrees
- moved R15 13.8 mm to (66.9, 69.3), turned to -90 degrees
- moved R9 13.1 mm to (51.8, 70.1), turned to 180 degrees
- moved R22 13.1 mm to (59.1, 60.5), turned to 180 degrees
- moved R10 13.0 mm to (55.2, 78.3), turned to -90 degrees
- moved R8 12.7 mm to (56.3, 75.5), turned to 180 degrees
- moved R20 10.8 mm to (54.5, 65.5)
- moved R6 10.6 mm to (63.7, 86.5), turned to 0 degrees
- moved C5 10.4 mm to (55.2, 81.6)
- moved C3 10.3 mm to (58.0, 86.8)
- moved R11 10.3 mm to (54.3, 86.8)
- moved C12 10.3 mm to (64.9, 67.2)
- moved R17 10.3 mm to (64.9, 62.8)
- moved C8 10.3 mm to (66.9, 62.8)
- moved C9 10.3 mm to (55.1, 63.0)
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Connections:
- R12 pad 2: Net-(J12-Pin_3) -> (no net)
- R14 pad 2: Net-(J12-Pin_4) -> (no net)
- R16 pad 1: Net-(J7-Pin_1) -> (no net)
- R21 pad 2: Net-(J12-Pin_5) -> (no net)
- R22 pad 1: Net-(J7-Pin_2) -> (no net)
- R5 pad 1: Net-(J7-Pin_3) -> (no net)
- R8 pad 2: Net-(J12-Pin_2) -> (no net)
- R9 pad 1: Net-(J7-Pin_4) -> (no net)
- U1 pad 10: Net-(J7-Pin_4) -> (no net)
- U1 pad 3: Net-(J7-Pin_3) -> (no net)
Routing:
- net (no net): track 0.00 -> 190.9 mm
- net GND: track 92.8 -> 211.1 mm, vias 0 -> 1
- net Net-(J7-Pin_2): track 30.4 -> 0.00 mm
- net Net-(J7-Pin_4): track 27.1 -> 0.00 mm
- net Net-(J7-Pin_3): track 17.4 -> 0.00 mm
- net Net-(U2D--): track 24.0 -> 8.79 mm
- net Net-(J12-Pin_3): track 12.8 -> 0.00 mm
- net +12V: track 25.0 -> 34.9 mm, vias 1 -> 2
- net Net-(J12-Pin_4): track 9.43 -> 0.00 mm
- net -12V: track 25.2 -> 33.6 mm, vias 1 -> 2
- net Net-(J12-Pin_2): track 7.25 -> 0.00 mm
- net Net-(U1B--): track 17.4 -> 24.2 mm
- net Net-(C7-Pad2): track 12.6 -> 6.55 mm
- net Net-(J7-Pin_1): track 5.86 -> 0.00 mm
- net Net-(U1D--): track 22.5 -> 18.7 mm
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Other:
- board size 20 x 27.8 mm -> 20 x 48.2 mm
- board text added: "Loop v1.0"
- board text added: "Serial"
- board text added: "by Geir & Adam"
- board text added: "https://github.com/GugeNet/Loop"

Commit message: Leveller 1.0b
Parts:
- moved R22 3.89 mm to (63.0, 60.2)
- moved J6 3.73 mm to (58.0, 55.4)
- moved D1 2.99 mm to (59.1, 57.9)
- moved FB1 2.49 mm to (59.2, 60.2)
- moved R13 2.03 mm to (64.9, 72.2)
- moved C10 2.03 mm to (59.0, 72.2)
- moved C12 2.03 mm to (66.9, 66.8)
- moved C3 2.03 mm to (60.0, 86.5)
- moved C4 2.03 mm to (65.0, 43.9)
- moved C6 2.03 mm to (65.0, 50.8)
- moved C9 2.03 mm to (57.1, 62.6)
- moved D4 2.03 mm to (68.8, 51.7)
- moved J13 2.03 mm to (54.5, 79.1)
- moved J14 2.03 mm to (69.5, 79.1)
- moved J17 2.03 mm to (53.8, 41.8)
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Routing:
- net -12V: track 33.6 -> 30.6 mm
- net (no net): track 190.9 -> 188.0 mm
- net Net-(C9-Pad1): track 6.79 -> 8.73 mm
- net GND: track 211.1 -> 210.4 mm
Other:
- board text added: "Loop v1.0b"
- board text removed: "Loop v1.0"

Commit message: HW 1.0c
Parts:
- removed J13: Audio to Daisy, connect to J13, Connector_PinHeader_2.54mm:PinHeader_1x03_P2.54mm_Vertical
- removed J14: Audio from Daisy, connect to J10, Connector_PinHeader_2.54mm:PinHeader_1x03_P2.54mm_Vertical
- removed J17: Audio output, connect to J16, Connector_PinHeader_2.54mm:PinHeader_1x03_P2.54mm_Vertical
- removed J18: Audio input, connect to J15, Connector_PinHeader_2.54mm:PinHeader_1x03_P2.54mm_Vertical
- removed R11: 10K, Resistor_SMD:R_0603_1608Metric
- added C13: 560pF, Capacitor_SMD:C_0603_1608Metric, F.Cu at (58.2, 59.1)
- added C14: 47pF, Capacitor_SMD:C_0603_1608Metric, F.Cu at (67.9, 73.2)
- added J7: Conn_01x05, Connector_PinHeader_2.54mm:PinHeader_1x05_P2.54mm_Vertical, F.Cu at (72.3, 66.7)
- added J8: Conn_01x05, Connector_PinHeader_2.54mm:PinHeader_1x05_P2.54mm_Vertical, F.Cu at (57.2, 66.7)
- added MOUNT1: MountingHole_2.7mm_M2.5, MountingHole:MountingHole_2.7mm_M2.5, F.Cu at (64.7, 50.3)
- added R23: 100K, Resistor_SMD:R_0603_1608Metric, F.Cu at (63.0, 72.9)
- added R24: 100K, Resistor_SMD:R_0603_1608Metric, F.Cu at (67.9, 71.3)
- added R25: 100K, Resistor_SMD:R_0603_1608Metric, F.Cu at (70.1, 83.6)
- C2: value 560pF -> 47pF
- R5: value 2M -> 10K
- R9: value 2M -> 100K
- moved C9 21.1 mm to (59.2, 83.6), turned to 90 degrees
- moved C3 18.9 mm to (63.0, 67.7)
- moved FB1 18.1 mm to (56.5, 42.3), turned to -90 degrees
- moved R12 17.2 mm to (73.4, 83.6), turned to 90 degrees
- moved R9 15.5 mm to (60.9, 83.6), turned to -90 degrees
- moved R18 15.5 mm to (69.4, 68.8)
- moved J6 14.0 mm to (59.6, 41.5), turned to -90 degrees
- moved C7 13.9 mm to (71.2, 59.1)
- moved R13 13.8 mm to (69.5, 59.1)
- moved R16 13.7 mm to (56.6, 59.1), turned to 90 degrees
- moved C8 13.7 mm to (62.9, 74.7), turned to 180 degrees
- moved FB2 13.6 mm to (73.0, 42.3), turned to -90 degrees
- moved R14 13.4 mm to (59.9, 59.1)
- moved R15 13.0 mm to (64.7, 56.7), turned to 0 degrees
- moved C10 12.3 mm to (69.4, 65.6), turned to 90 degrees
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Connections:
- C10 pad 2: Net-(U2D--) -> Net-(U2A--)
- C2 pad 1: Net-(U1B--) -> (no net)
- C2 pad 2: Net-(C2-Pad2) -> Net-(U1A--)
- C3 pad 1: Net-(U1D--) -> Net-(U2D--)
- C4 pad 1: (no net) -> +12V
- C6 pad 2: (no net) -> -12V
- C7 pad 1: Net-(U2A--) -> Net-(U2B--)
- C8 pad 1: Net-(C8-Pad1) -> Net-(U1C--)
- C8 pad 2: Net-(U2B--) -> (no net)
- C9 pad 2: Net-(U2C--) -> Net-(U1D--)
- D1 pad 2: (no net) -> -12V
- D4 pad 1: (no net) -> +12V
- FB1 pad 1: -12V -> (no net)
- FB2 pad 1: +12V -> (no net)
- R10 pad 1: Net-(U1C--) -> Net-(C9-Pad1)
- R10 pad 2: Net-(U1D--) -> Net-(U1A--)
- R12 pad 1: Net-(C3-Pad2) -> (no net)
- R13 pad 1: Net-(U2A--) -> Net-(U2B--)
- R14 pad 1: Net-(U2A--) -> (no net)
- R14 pad 2: (no net) -> Net-(U2C--)
- R15 pad 1: Net-(U2B--) -> Net-(U2C--)
- R16 pad 2: Net-(C8-Pad1) -> (no net)
- R17 pad 1: Net-(C8-Pad1) -> Net-(U2B--)
- R17 pad 2: Net-(U2B--) -> (no net)
- R18 pad 1: Net-(C9-Pad1) -> Net-(U2A--)
- R18 pad 2: Net-(U2C--) -> (no net)
- R19 pad 2: Net-(U2D--) -> Net-(U2A--)
- R20 pad 1: Net-(U2C--) -> Net-(U2D--)
- R21 pad 1: Net-(U2D--) -> Net-(C3-Pad2)
- R21 pad 2: (no net) -> Net-(U2D--)
- R22 pad 2: Net-(C9-Pad1) -> Net-(C3-Pad2)
- R5 pad 1: (no net) -> Net-(U1D--)
- R5 pad 2: GND -> (no net)
- R6 pad 1: Net-(U1A--) -> (no net)
- R7 pad 1: Net-(U1B--) -> (no net)
- R7 pad 2: Net-(C2-Pad2) -> Net-(U1C--)
- R8 pad 1: Net-(C2-Pad2) -> (no net)
- R9 pad 1: (no net) -> Net-(U1D--)
- R9 pad 2: GND -> Net-(C9-Pad1)
- U1 pad 1: Net-(U1A--) -> (no net)
- U1 pad 10: (no net) -> GND
- U1 pad 14: Net-(C3-Pad2) -> Net-(C9-Pad1)
- U1 pad 3: (no net) -> GND
- U1 pad 7: Net-(C2-Pad2) -> (no net)
- U1 pad 8: Net-(U1C--) -> (no net)
- U2 pad 1: Net-(C7-Pad2) -> Net-(C10-Pad1)
- U2 pad 14: Net-(C10-Pad1) -> Net-(C3-Pad2)
- U2 pad 7: Net-(C8-Pad1) -> Net-(C7-Pad2)
- U2 pad 8: Net-(C9-Pad1) -> (no net)
Routing:
- net (no net): track 188.0 -> 87.1 mm
- net GND: track 210.4 -> 141.0 mm
- net Net-(U1B--): track 24.2 -> 8.98 mm
- net Net-(U1A--): track 3.45 -> 17.0 mm
- net Net-(U1D--): track 18.7 -> 5.50 mm
- net -12V: track 30.6 -> 42.0 mm, vias 2 -> 3
- net Net-(C2-Pad2): track 10.0 -> 0.00 mm
- net +12V: track 34.9 -> 44.9 mm, vias 2 -> 3
- net Net-(U1C--): track 3.72 -> 10.3 mm
- net Net-(C8-Pad1): track 6.57 -> 0.00 mm
- net Net-(C10-Pad1): track 12.1 -> 5.86 mm
- net Net-(U2B--): track 9.14 -> 5.62 mm
- net Net-(C9-Pad1): track 8.73 -> 5.64 mm
- net Net-(C3-Pad2): track 9.65 -> 7.09 mm
- net Net-(U2A--): track 8.26 -> 10.7 mm
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Other:
- board text added: "Loop v1.0c"
- board text removed: "Loop v1.0b"

Commit message: Version 1.0d hardware
Parts:
- removed J7: Conn_01x05, Connector_PinHeader_2.54mm:PinHeader_1x05_P2.54mm_Vertical
- added J10: Conn_01x06_Socket, Connector_PinHeader_2.54mm:PinHeader_1x06_P2.54mm_Vertical, F.Cu at (56.9, 74.8)
- moved C12 17.9 mm to (53.5, 59.5), turned to -90 degrees
- moved J8 16.7 mm to (40.6, 64.6)
- moved R17 16.5 mm to (56.9, 57.4)
- moved C1 16.3 mm to (55.8, 78.4), turned to 0 degrees
- moved R18 16.2 mm to (53.4, 66.1)
- moved R8 16.2 mm to (52.8, 72.2)
- moved U1 16.2 mm to (49.5, 77.6)
- moved R25 16.2 mm to (54.2, 80.9)
- moved U2 16.2 mm to (48.7, 59.6)
- moved C14 16.2 mm to (51.9, 70.5)
- moved C3 16.2 mm to (47.0, 65.1)
- moved D1 16.2 mm to (40.5, 44.0)
- moved D4 16.2 mm to (57.0, 44.0)
- moved R20 16.2 mm to (50.9, 66.7)
- moved R21 16.2 mm to (44.0, 62.9)
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Connections:
- C1 pad 1: GND -> (no net)
- C11 pad 2: GND -> (no net)
- C12 pad 1: GND -> (no net)
- C5 pad 2: GND -> (no net)
- J8 pad 1: GND -> (no net)
- U1 pad 10: GND -> (no net)
- U1 pad 12: GND -> (no net)
- U1 pad 3: GND -> (no net)
- U1 pad 5: GND -> (no net)
- U2 pad 10: GND -> (no net)
- U2 pad 12: GND -> (no net)
- U2 pad 3: GND -> (no net)
- U2 pad 5: GND -> (no net)
Routing:
- net GND: track 141.0 -> 72.4 mm
- net (no net): track 87.1 -> 154.9 mm, vias 0 -> 2
- net Net-(C3-Pad2): track 7.09 -> 6.59 mm
- net +12V: vias 3 -> 2
- added copper zone on B.Cu, net (none)
- added copper zone on F.Cu, net (none)
Other:
- board text added: "Loop v1.0d"
- board text removed: "Loop v1.0c"
