File: Hardware/PCB/Looper_main.kicad_pcb (KiCad board)
At the start: 2 copper layers, 20 x 110.1 mm, 28 parts, among them J1 Out right, J11 Conn_01x06_Pin, J2 In left, J3 Trig Loop, J4 Out left, J5 In right, J6 Eurorack_Power, J8 Conn_01x05_Socket

Commit message: Version 1.0 of hardware ordered
Parts:
- removed C4, C6: 10uF, Capacitor_SMD:CP_Elec_4x5.4
- removed D1, D4: 1N5819, Diode_SMD:D_SOD-123
- removed FB1, FB2: FerriteBead, Resistor_SMD:R_0603_1608Metric
- removed J11: Conn_01x06_Pin, Connector_PinHeader_2.54mm:PinHeader_1x06_P2.54mm_Vertical
- removed J6: Eurorack_Power, Connector_PinHeader_2.54mm:PinHeader_2x05_P2.54mm_Vertical
- removed J8: Conn_01x05_Socket, Connector_PinHeader_2.54mm:PinHeader_1x05_P2.54mm_Vertical
- added J10: Audio from Daisy, connect to J14, Connector_PinHeader_2.54mm:PinHeader_1x03_P2.54mm_Vertical, F.Cu at (-4.90, -98.5)
- added J15: Audio input, connect to J18, Connector_PinHeader_2.54mm:PinHeader_1x03_P2.54mm_Vertical, F.Cu at (-5.60, -135.8)
- added J16: Audio output, connect to J17, Connector_PinHeader_2.54mm:PinHeader_1x03_P2.54mm_Vertical, F.Cu at (10.8, -135.8)
- added J9: Audio to Daisy, connect to J13, Connector_PinHeader_2.54mm:PinHeader_1x03_P2.54mm_Vertical, F.Cu at (10.1, -98.5)
- moved D2 32.6 mm to (-4.45, -109.4)
- moved MOUNT1 27.5 mm to (-4.20, -30.6)
- moved J1 24.9 mm to (-2.40, -117.4)
- moved J4 24.9 mm to (-2.40, -130.4)
- moved J3 19.3 mm to (2.60, -104.0)
- moved S1 19.3 mm to (7.60, -91.4)
- moved S2 19.3 mm to (-2.40, -91.4)
- moved R1 19.3 mm to (2.55, -45.7)
- moved SW1 19.3 mm to (2.60, -78.9)
- moved SW2 19.3 mm to (2.60, -64.9)
- moved A1 19.3 mm to (10.2, -37.3)
- moved D3 19.3 mm to (-1.35, -42.4)
- moved R2 19.3 mm to (-2.50, -60.8)
- moved R3 19.3 mm to (-0.25, -71.8)
- moved R4 19.3 mm to (7.45, -41.5)
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Connections:
- J5 pad T: In Right -> (no net)
Routing:
- net GND: track 236.9 -> 278.1 mm, vias 0 -> 2
- net -12V: track 29.1 -> 0.00 mm
- net (no net): track 0.00 -> 26.3 mm
- net Net-(D1-A): track 21.9 -> 0.00 mm
- net In Left: track 29.6 -> 43.6 mm
- net Out Right: track 18.1 -> 31.9 mm
- net Out_R: track 17.5 -> 30.2 mm
- net Net-(D4-K): track 11.2 -> 0.00 mm
- net Net-(D4-A): track 10.4 -> 0.00 mm
- net In Right: track 7.79 -> 0.00 mm
- net Net-(A1-AUDIO_IN_L): track 34.5 -> 27.3 mm
- net Net-(A1-AUDIO_OUT_L): track 23.1 -> 29.8 mm
- net Net-(A1-ADC_INP10): track 87.3 -> 93.6 mm
- net Out Left: track 39.1 -> 43.7 mm
- net Net-(D1-K): track 2.42 -> 0.00 mm
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
Commit message: HW 1.0c
Parts:
- removed D2, D3: 1N5819, Diode_SMD:D_SOD-123
- removed J10: Audio from Daisy, connect to J14, Connector_PinHeader_2.54mm:PinHeader_1x03_P2.54mm_Vertical
- removed J15: Audio input, connect to J18, Connector_PinHeader_2.54mm:PinHeader_1x03_P2.54mm_Vertical
- removed J16: Audio output, connect to J17, Connector_PinHeader_2.54mm:PinHeader_1x03_P2.54mm_Vertical
- removed J9: Audio to Daisy, connect to J13, Connector_PinHeader_2.54mm:PinHeader_1x03_P2.54mm_Vertical
- removed the MOUNT1 at (-4.20, -30.6)
- added J11: Conn_01x05, Connector_PinHeader_2.54mm:PinHeader_1x05_P2.54mm_Vertical, F.Cu at (92.4, 73.8)
- added J12: Conn_01x05, Connector_PinHeader_2.54mm:PinHeader_1x05_P2.54mm_Vertical, F.Cu at (107.6, 73.8)
- added MOUNT1: MountingHole_2.7mm_M2.5, MountingHole:MountingHole_2.7mm_M2.5, F.Cu at (100.0, 57.3)
- added MOUNT1: MountingHole_2.7mm_M2.5, MountingHole:MountingHole_2.7mm_M2.5, F.Cu at (93.2, 150.6)
- added Q1: MMBT3904, Package_TO_SOT_SMD:SOT-23, F.Cu at (103.6, 76.1)
- added R11: 100K, Resistor_SMD:R_0603_1608Metric, F.Cu at (103.6, 72.4)
- added R26: 10K, Resistor_SMD:R_0603_1608Metric, F.Cu at (95.7, 83.6)
- added R27: 1K, Resistor_SMD:R_0603_1608Metric, F.Cu at (95.6, 95.2)
- added R29: 100K, Resistor_SMD:R_0603_1608Metric, F.Cu at (107.9, 70.9)
- moved R1 206.5 mm to (98.4, 137.2), turned to 180 degrees
- moved A1 205.7 mm to (107.6, 143.9)
- moved J3 205.7 mm to (100.0, 77.2)
- moved S1 205.7 mm to (105.0, 89.8)
- moved S2 205.7 mm to (95.0, 89.8)
- moved SW1 205.7 mm to (100.0, 102.3)
- moved SW2 205.7 mm to (100.0, 116.3)
- moved J1 205.7 mm to (95.0, 63.8)
- moved J2 205.7 mm to (105.0, 50.8)
- moved J4 205.7 mm to (95.0, 50.8)
- moved J5 205.7 mm to (105.0, 63.8)
- moved SW3 205.7 mm to (99.9, 130.3)
- moved SW4 205.7 mm to (100.0, 144.3)
- moved R4 204.8 mm to (104.6, 138.8), turned to 180 degrees
- moved R2 204.4 mm to (94.9, 119.0)
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Connections:
- A1 pad 14: Net-(A1-USART1_TX) -> (no net)
- A1 pad 15: Net-(A1-USART1_RX) -> (no net)
- A1 pad 16: Net-(A1-AUDIO_IN_L) -> (no net)
- A1 pad 17: Net-(A1-AUDIO_IN_R) -> (no net)
- A1 pad 18: Net-(A1-AUDIO_OUT_L) -> (no net)
- A1 pad 19: Out_R -> (no net)
- A1 pad 2: Net-(A1-SDMMC1_D3) -> (no net)
- A1 pad 22: Net-(A1-ADC_INP10) -> (no net)
- A1 pad 23: unconnected-(A1-ADC_INP15-Pad23) -> (no net)
- A1 pad 24: unconnected-(A1-ADC_INP5-Pad24) -> (no net)
- A1 pad 25: unconnected-(A1-ADC_INP7-Pad25) -> (no net)
- A1 pad 26: unconnected-(A1-ADC_INP3-Pad26) -> (no net)
- A1 pad 27: Net-(A1-ADC_INP11) -> (no net)
- A1 pad 28: Net-(A1-ADC1_INP4) -> (no net)
- A1 pad 29: Net-(A1-DAC1_OUT2) -> (no net)
- A1 pad 3: Net-(A1-SDMMC1_D2) -> (no net)
- A1 pad 30: Net-(A1-DAC1_OUT1) -> (no net)
- A1 pad 31: Net-(A1-SAI2_MCLK_B) -> (no net)
- A1 pad 32: Net-(A1-SAI2_SD_B) -> (no net)
- A1 pad 33: Net-(A1-SAI2_SD_A) -> (no net)
- A1 pad 34: Net-(A1-SAI2_FS_B) -> (no net)
- A1 pad 35: Net-(A1-SAI2_SCK_B) -> (no net)
- A1 pad 4: Net-(A1-SDMMC1_D1) -> (no net)
- J1 pad TN: Out Left -> GND
- J3 pad T: Net-(A1-ADC_INP10) -> (no net)
- J5 pad TN: In Left -> GND
- R1 pad 1: Net-(A1-SAI2_SCK_B) -> (no net)
- R1 pad 2: Net-(R1-Pad2) -> (no net)
- R2 pad 1: Net-(R2-Pad1) -> (no net)
- R2 pad 2: Net-(A1-SAI2_SD_B) -> (no net)
- R3 pad 2: Net-(A1-ADC1_INP4) -> (no net)
- R4 pad 1: Net-(A1-SDMMC1_D2) -> (no net)
- S1 pad 1: Net-(A1-USART1_RX) -> (no net)
- S2 pad 1: Net-(A1-USART1_TX) -> (no net)
- SW1 pad 1: Net-(A1-DAC1_OUT2) -> (no net)
- SW1 pad 3: Net-(A1-ADC_INP11) -> (no net)
- SW2 pad 2: Net-(A1-SAI2_MCLK_B) -> (no net)
- SW2 pad 3: Net-(R2-Pad1) -> (no net)
- SW2 pad 4: Net-(A1-DAC1_OUT1) -> (no net)
- SW3 pad 1: Net-(A1-SAI2_FS_B) -> (no net)
- SW3 pad 3: Net-(A1-SAI2_SD_A) -> (no net)
- SW3 pad 4: Net-(R1-Pad2) -> (no net)
- SW4 pad 1: Net-(A1-SDMMC1_D3) -> (no net)
- SW4 pad 3: Net-(A1-SDMMC1_D1) -> (no net)
Routing:
- net (no net): track 26.3 -> 329.8 mm
- net Net-(A1-ADC_INP10): track 93.6 -> 0.00 mm
- net +3.3V: track 2.02 -> 55.8 mm, vias 0 -> 1
- net GND: track 278.1 -> 224.9 mm, vias 2 -> 0
- net Net-(A1-USART1_TX): track 33.7 -> 0.00 mm
- net Net-(A1-USART1_RX): track 30.8 -> 0.00 mm
- net Out_R: track 30.2 -> 0.00 mm
- net Net-(A1-AUDIO_OUT_L): track 29.8 -> 0.00 mm
- net Net-(A1-AUDIO_IN_R): track 28.7 -> 0.00 mm
- net Net-(A1-AUDIO_IN_L): track 27.3 -> 0.00 mm
- net Net-(A1-DAC1_OUT2): track 17.9 -> 0.00 mm
- net Net-(A1-SAI2_MCLK_B): track 16.1 -> 0.00 mm
- net Net-(A1-SDMMC1_D1): track 14.0 -> 0.00 mm
- net Net-(A1-DAC1_OUT1): track 13.2 -> 0.00 mm
- net Out Right: track 31.9 -> 19.3 mm
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
Commit message: Version 1.0d hardware
Parts:
- removed J11: Conn_01x05, Connector_PinHeader_2.54mm:PinHeader_1x05_P2.54mm_Vertical
- removed the MOUNT1 at (100.0, 57.3)
- removed the MOUNT1 at (93.2, 150.6)
- added J9: Conn_01x06_Pin, Connector_PinHeader_2.54mm:PinHeader_1x06_P2.54mm_Vertical, F.Cu at (56.2, 84.4)
- added MOUNT1: MountingHole_2.7mm_M2.5, MountingHole:MountingHole_2.7mm_M2.5, F.Cu at (64.3, 57.2)
- added MOUNT1: MountingHole_2.7mm_M2.5, MountingHole:MountingHole_2.7mm_M2.5, F.Cu at (57.5, 150.5)
- moved R29 48.4 mm to (60.1, 78.5), turned to 90 degrees
- moved SW3 35.7 mm to (64.2, 130.2)
- moved R1 35.7 mm to (62.6, 137.1)
- moved R2 35.7 mm to (59.2, 118.9)
- moved R26 35.7 mm to (60.0, 83.5)
- moved A1 35.7 mm to (71.9, 143.8)
- moved J1 35.7 mm to (59.3, 63.7)
- moved J2 35.7 mm to (69.3, 50.7)
- moved J3 35.7 mm to (64.3, 77.1)
- moved J4 35.7 mm to (59.3, 50.7)
- moved J5 35.7 mm to (69.3, 63.7)
- moved Q1 35.7 mm to (67.9, 76.0)
- moved R11 35.7 mm to (67.9, 72.3)
- moved R27 35.7 mm to (59.8, 95.1)
- moved R4 35.7 mm to (68.9, 138.7)
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Connections:
- A1 pad 20: GND -> (no net)
- J1 pad S: GND -> (no net)
- J1 pad TN: GND -> (no net)
- J12 pad 1: GND -> (no net)
- J2 pad S: GND -> (no net)
- J2 pad TN: GND -> (no net)
- J4 pad S: GND -> (no net)
- J4 pad TN: GND -> (no net)
- J5 pad S: GND -> (no net)
- J5 pad TN: GND -> (no net)
Routing:
- net (no net): track 329.8 -> 416.6 mm
- net GND: track 224.9 -> 151.5 mm
- net +12V: track 74.1 -> 60.9 mm
- net Out Left: track 41.3 -> 33.3 mm
- net Out Right: track 19.3 -> 12.0 mm
- net In Left: track 41.6 -> 36.4 mm
- net Net-(R3-Pad1): track 10.8 -> 7.24 mm
- added copper zone on B.Cu, net (none)
- added copper zone on F.Cu, net (none)
